Commit message: initial package

File: src/m2wr_description/urdf/rover.xacro (robot description, xacro)
@@ -102,5 +102,5 @@
      <origin rpy=" 0 0 0" xyz="0.065 0 -0.025"/>
       <geometry>
-        <cylinder length="0.01" radius="0.0025"/>
+        <cylinder length="0.0075" radius="0.0025"/>
       </geometry>
       <surface>
@@ -118,5 +118,5 @@
       <origin rpy="0 0 0" xyz="0.065 0 -0.025"/>
       <geometry>
-        <cylinder length="0.01" radius="0.0025"/>
+        <cylinder length="0.0075" radius="0.0025"/>
       </geometry>
       <material name="blue"/>
@@ -126,5 +126,5 @@
      <origin rpy=" 0 0 0" xyz="-0.065 0 -0.025"/>
       <geometry>
-        <cylinder length="0.01" radius="0.0025"/>
+        <cylinder length="0.0075" radius="0.0025"/>
       </geometry>
       <surface>
@@ -142,5 +142,5 @@
       <origin rpy="0 0 0" xyz="-0.065 0 -0.025"/>
       <geometry>
-        <cylinder length="0.01" radius="0.0025"/>
+        <cylinder length="0.0075" radius="0.0025"/>
       </geometry>
       <material name="blue"/>
@@ -157,6 +157,6 @@
             <mu>0</mu>
             <mu2>0</mu2>
-            <slip1>1.0</slip1>
-            <slip2>1.0</slip2>
+            <slip1>0.0</slip1>
+            <slip2>0.0</slip2>
           </ode>
         </friction>
@@ -180,6 +180,6 @@
             <mu>0</mu>
             <mu2>0</mu2>
-            <slip1>1.0</slip1>
-            <slip2>1.0</slip2>
+            <slip1>0.0</slip1>
+            <slip2>0.0</slip2>
           </ode>
         </friction>

Commit message: initial package

File: src/m2wr_description/urdf/rover.xacro (robot description, xacro)
@@ -69,5 +69,5 @@
         <frameName>camera_link</frameName>
         <hackBaseline>0.07</hackBaseline>
-        <distortionK1>0.0</distortionK1>5
+        <distortionK1>0.0</distortionK1>
         <distortionK2>0.0</distortionK2>
         <distortionK3>0.0</distortionK3>
@@ -268,5 +268,5 @@
   </link>
   <joint name="camera_joint" type="fixed">
-	    <origin xyz="0.07 0 0.05" rpy="0 0 0"/>
+	    <origin xyz="0.085 0 0.05" rpy="0 1.0466 0"/>
 	    <child link="camera_link"/>
 	    <parent link="link_chassis"/>
